Commit message: pddls

File: assets/models/Faucet/14/mobility.urdf (robot description, URDF)
Before this commit: robot partnet_2781a072e2645ccdedf1aa83ea962bc0, 5 links, 4 joints
Links:
- added link link_nob_0; collision mesh filename=faucet_objs/new-11.obj; visual mesh filename=faucet_objs/new-11.obj
- added link link_nob_1; collision mesh filename=faucet_objs/new-7.obj; visual mesh filename=faucet_objs/new-7.obj
- added link link_nob_2; visual mesh filename=faucet_objs/new-14.obj
- added link tube_head; collision mesh filename=faucet_objs/new-1.obj; visual mesh filename=faucet_objs/new-1.obj
- link link_2: geometry collision mesh filename=faucet_objs/new-0.obj; collision mesh filename=faucet_objs/original-3.obj
- link link_3: geometry collision mesh filename=faucet_objs/new-12.obj; collision mesh filename=faucet_objs/new-8.obj
Joints:
- added joint joint_head: type fixed, parent link_3, child tube_head, origin xyz=0.004107500000000028 0 -0.0790015, axis 0 1 0
- added joint joint_nob_0: type fixed, parent link_3, child link_nob_0, origin xyz=0 0 0, axis 0 1 0
- added joint joint_nob_1: type fixed, parent link_3, child link_nob_1, origin xyz=0 0 0, axis 0 1 0
- added joint joint_nob_2: type fixed, parent link_3, child link_nob_2, origin xyz=0 0 0, axis 0 1 0
- joint joint_faucet_0: parent link_3 -> link_nob_0
- joint joint_faucet_1: parent link_3 -> link_nob_1
- joint joint_faucet_2: parent link_3 -> link_nob_2; type continuous -> fixed

File: assets/models/Fridge/10144/mobility.urdf (robot description, URDF)
Before this commit: robot partnet_9e53ec8bedae98859807c66948157e66, 6 links, 5 joints
Links:
- added link fridge_collision_bottom_link; collision mesh filename=textured_objs/fridge_body_bottom.obj; visual mesh filename=textured_objs/fridge_body_bottom.obj
- added link fridge_collision_left_link; collision mesh filename=textured_objs/fridge_body_left.obj; visual mesh filename=textured_objs/fridge_body_left.obj
- added link fridge_collision_right_link; collision mesh filename=textured_objs/fridge_body_right.obj; visual mesh filename=textured_objs/fridge_body_right.obj
- added link fridge_collision_top_link; collision mesh filename=textured_objs/fridge_body_top.obj; visual mesh filename=textured_objs/fridge_body_top.obj
- link fridge_body: geometry visual mesh filename=textured_objs/original-119.obj; visual mesh filename=textured_objs/original-122.obj
Joints:
- added joint fridge_collision_bottom: type fixed, parent fridge_body, child fridge_collision_bottom_link, origin xyz=0 0 0
- added joint fridge_collision_left: type fixed, parent fridge_body, child fridge_collision_left_link, origin xyz=0 0 0
- added joint fridge_collision_right: type fixed, parent fridge_body, child fridge_collision_right_link, origin xyz=0 0 0
- added joint fridge_collision_top: type fixed, parent fridge_body, child fridge_collision_top_link, origin xyz=0 0 0

File: assets/models/Oven/01909/mobility.urdf (robot description, URDF)
Before this commit: robot partnet_8295e45a734c059d1f3d773b4af1f0c9, 7 links, 6 joints
Links:
- added link knob_link_2; collision mesh filename=textured_objs/original-10.obj; visual mesh filename=textured_objs/original-10.obj
- link link_2: geometry collision mesh filename=textured_objs/original-51.obj; visual mesh filename=textured_objs/original-51.obj
Joints:
- removed joint joint_1
- removed joint joint_2
- removed joint joint_3
- removed joint joint_4
- added joint knob_button_2: type fixed, parent link_5, child link_2, origin xyz=0.2262559467393136 0.7720745754611937 -0.15151306153341626, axis 0 0.19256852863983123 0.9812835277214688
- added joint knob_joint_1: type revolute, parent link_5, child link_1, origin xyz=0.41708094673931356 0.7720745754611937 -0.15151306153341626, axis 0 0.19256852863983123 0.9812835277214688, limit lower=-0.0 upper=1.046666667
- added joint knob_joint_2: type revolute, parent link_2, child knob_link_2, origin xyz=0 0 0, axis 0 0.19256852863983123 0.9812835277214688, limit lower=-0.0 upper=1.046666667
- added joint knob_joint_3: type revolute, parent link_5, child link_3, origin xyz=-0.15347888005765334 0.7720745754611937 -0.15151306153341626, axis 0 0.19256852863983126 0.9812835277214688, limit lower=-0.0 upper=5.672320068981571
- added joint knob_joint_4: type revolute, parent link_5, child link_4, origin xyz=-0.3520335 0.7720735939143407 -0.15153806521756305, axis 0 0.1925993712652328 0.9812774746157363, limit lower=-6.283185307179586 upper=-0.6108652381980153

File: assets/models/counter/urdf/kitchen_part_right_gen_convex.urdf (robot description, URDF)
Before this commit: robot kitchen_part_right, 57 links, 56 joints
Links:
- removed link back_left_knob
- removed link back_right_knob
- removed link front_left_knob
- removed link front_right_knob
Joints:
- removed joint back_left_knob_transform
- removed joint back_right_knob_transform
- removed joint front_left_knob_transform
- removed joint front_right_knob_transform
