Commit message: make demo gifs

File: assets/models/Dishwasher/2085/mobility.urdf (robot description, URDF)
Before this commit: robot partnet_185cf76909e948f0fa80fb391ee7ccee, 5 links, 4 joints
Links:
- added link handle_link; collision mesh filename=textured_objs/new-2.obj; visual mesh filename=textured_objs/new-2.obj
- added link upper_shelf; collision mesh filename=textured_objs/original-4-bottom.obj; collision mesh filename=textured_objs/original-4-left.obj
- link link_0: geometry collision mesh filename=textured_objs/new-0.obj; collision mesh filename=textured_objs/new-1-back.obj
- link link_1: geometry collision mesh filename=textured_objs/new-3.obj; collision mesh filename=textured_objs/new-4.obj
Joints:
- added joint handle_joint: type fixed, parent link_1, child handle_link, origin xyz=0 0 0
- added joint upper_shelf_joint: type fixed, parent link_1, child upper_shelf, origin xyz=0 0 0
