Commit message: fixed wconf poses assign problem

File: assets/models/Basin/102379/mobility.urdf (robot description, URDF)
Before this commit: robot partnet_3ac64751-e075-488d-9938-9123dc88b2b6-0, 5 links, 4 joints
Links:
- added link link_collision_1; collision mesh filename=textured_objs/basin-minus-y.obj; visual mesh filename=textured_objs/basin-minus-y.obj
- added link link_collision_2; collision mesh filename=textured_objs/basin-minus-x.obj; visual mesh filename=textured_objs/basin-minus-x.obj
- added link link_collision_3; collision mesh filename=textured_objs/basin-plus-y.obj; visual mesh filename=textured_objs/basin-plus-y.obj
- added link link_collision_4; collision mesh filename=textured_objs/basin-plus-x.obj; visual mesh filename=textured_objs/basin-plus-x.obj
- link basin: geometry visual mesh filename=textured_objs/original-47.obj; visual mesh filename=textured_objs/original-48.obj
- link basin_bottom: geometry collision box size=1.26 .001 .84; visual box size=1.26 .001 .84
Joints:
- added joint joint_collision_1: type fixed, parent basin, child link_collision_1, origin xyz=0 0 0 rpy=0 0 0
- added joint joint_collision_2: type fixed, parent basin, child link_collision_2, origin xyz=0 0 0 rpy=0 0 0
- added joint joint_collision_3: type fixed, parent basin, child link_collision_3, origin xyz=0 0 0 rpy=0 0 0
- added joint joint_collision_4: type fixed, parent basin, child link_collision_4, origin xyz=0 0 0 rpy=0 0 0
