Commit message: fridge model fixes

File: assets/models/Fridge/10144/mobility.urdf (robot description, URDF)
Before this commit: robot partnet_9e53ec8bedae98859807c66948157e66, 10 links, 9 joints
Links:
- added link fridge_collision_back_link; collision mesh filename=textured_objs/fridge_body_back.obj; visual mesh filename=textured_objs/fridge_body_back.obj
- link door_frame: geometry collision mesh filename=textured_objs/original-123.obj; collision mesh filename=textured_objs/original-124.obj
- link fridge_door_handle: geometry collision mesh filename=textured_objs/handle_grasp-new.obj; visual mesh filename=textured_objs/handle_grasp-new.obj
Joints:
- added joint fridge_collision_back: type fixed, parent fridge_body, child fridge_collision_back_link, origin xyz=0 0 0
