Commit message: Debug reading urdf

File: assets/models/counter/urdf/kitchen_part_right_gen_convex.urdf (robot description, URDF)
Before this commit: robot kitchen_part_right, 57 links, 56 joints
Links:
- link indigo_drawer_bottom: geometry collision box size=0.004 0.699 0.086; collision box size=0.511 0.004 0.086
- link indigo_drawer_top: geometry collision box size=0.004 0.699 0.086; collision box size=0.511 0.004 0.086

Commit message: pick in cabinet working

File: assets/models/counter/urdf/kitchen_part_right_gen_convex.urdf (robot description, URDF)
Before this commit: robot kitchen_part_right, 53 links, 52 joints
Links:
- link indigo_drawer_bottom: geometry collision box size=0.004 0.699 0.086; collision box size=0.511 0.004 0.086
- link indigo_drawer_top: geometry collision box size=0.004 0.699 0.086; collision box size=0.511 0.004 0.086
- link sektion: geometry collision mesh filename=package://counter/meshes/obj/sektion_top_three_new3_two.obj scale=1.0 1.0 1.0; visual mesh filename=package://counter/meshes/obj/sektion_top_three_new3_two.obj scale=1.0 1.0 1.0

Commit message: grasp & pose sampling

File: assets/models/counter/urdf/kitchen_part_right_gen_convex.urdf (robot description, URDF)
Before this commit: robot kitchen_part_right, 53 links, 52 joints
Links:
- link dagger: geometry collision mesh filename=package://counter/meshes/obj/sektion_top_two_glass_new.obj scale=1.0 1.0 1.0; visual mesh filename=package://counter/meshes/obj/sektion_top_two_glass_new.obj scale=1.0 1.0 1.0

Commit message: Updates

File: assets/models/counter/urdf/kitchen_part_right_gen_convex.urdf (robot description, URDF)
Before this commit: robot kitchen_part_right, 57 links, 56 joints
Links:
- removed link walls
- added link wall_back, mass 10.0; collision mesh filename=package://counter/meshes/obj/wall_back.obj scale=1.0 1.0 1.0; visual mesh filename=package://counter/meshes/obj/wall_back.obj scale=1.0 1.0 1.0
- added link wall_right, mass 10.0; collision mesh filename=package://counter/meshes/obj/wall_right.obj scale=1.0 1.0 1.0; visual mesh filename=package://counter/meshes/obj/wall_right.obj scale=1.0 1.0 1.0
Joints:
- removed joint wall_transform
- added joint wall_back_transform: type fixed, parent sektion, child wall_back, origin xyz=0 0 0 rpy=0 0 0
- added joint wall_right_transform: type fixed, parent sektion, child wall_right, origin xyz=0 0 0 rpy=0 0 0
