Commit message: added test cases

File: assets/models/Oven/01909/mobility.urdf (robot description, URDF)
Before this commit: robot partnet_8295e45a734c059d1f3d773b4af1f0c9, 8 links, 7 joints
Joints:
- joint joint_5: origin xyz=0.22 0 -0.45 rpy=1.570796326794897 0 -1.570796326794897 -> xyz=0.22 0 -0.3 rpy=1.570796326794897 0 -1.570796326794897

Commit message: Updates

File: assets/models/Oven/01909/mobility.urdf (robot description, URDF)
Before this commit: robot partnet_8295e45a734c059d1f3d773b4af1f0c9, 7 links, 6 joints
Links:
- added link knob_link_2; collision mesh filename=textured_objs/original-10.obj; visual mesh filename=textured_objs/original-10.obj
- link link_2: geometry collision mesh filename=textured_objs/original-51.obj; visual mesh filename=textured_objs/original-51.obj
Joints:
- removed joint joint_1
- removed joint joint_2
- removed joint joint_3
- removed joint joint_4
- added joint knob_button_2: type fixed, parent link_5, child link_2, origin xyz=0.2262559467393136 0.7720745754611937 -0.15151306153341626, axis 0 0.19256852863983123 0.9812835277214688
- added joint knob_joint_1: type revolute, parent link_5, child link_1, origin xyz=0.41708094673931356 0.7720745754611937 -0.15151306153341626, axis 0 0.19256852863983123 0.9812835277214688, limit lower=-0.0 upper=1.046666667
- added joint knob_joint_2: type revolute, parent link_2, child knob_link_2, origin xyz=0 0 0, axis 0 0.19256852863983123 0.9812835277214688, limit lower=-0.0 upper=1.046666667
- added joint knob_joint_3: type revolute, parent link_5, child link_3, origin xyz=-0.15347888005765334 0.7720745754611937 -0.15151306153341626, axis 0 0.19256852863983126 0.9812835277214688, limit lower=-0.0 upper=5.672320068981571
- added joint knob_joint_4: type revolute, parent link_5, child link_4, origin xyz=-0.3520335 0.7720735939143407 -0.15153806521756305, axis 0 0.1925993712652328 0.9812774746157363, limit lower=-6.283185307179586 upper=-0.6108652381980153
- joint joint_5: origin xyz=0.22 0 -0.45 rpy=1.570796326794897 0 -1.570796326794897 -> xyz=0.22 0 -0.3 rpy=1.570796326794897 0 -1.570796326794897
