Commit message: fridge modifications

File: assets/models/MiniFridge/11709/mobility.urdf (robot description, URDF)
Before this commit: robot partnet_f71397f01cab21ffaff7331733d1f0f5, 5 links, 4 joints
Links:
- link link_3: geometry collision mesh filename=textured_objs/original-1.obj; collision mesh filename=textured_objs/original-128.obj

File: assets/models/MiniFridge/12249/mobility.urdf (robot description, URDF)
Before this commit: robot partnet_3158fd17e409d38a732208e596b26ebc, 3 links, 2 joints
Links:
- added link handle; collision mesh filename=textured_objs/original-2-new.obj; visual mesh filename=textured_objs/original-2-new.obj
Joints:
- added joint joint_handle: type fixed, parent link_0, child handle, origin xyz=0 0 0.04, axis 0 0.9999999999999999 0
